Commit message: Edited urdfs

File: urdf/test/urdf/joint3.urdf (robot description, URDF)
Before this commit: robot single_leg, 6 links, 5 joints
Links:
- removed link FL_wheel
Joints:
- removed joint FL_wheel_axis
- joint FL_HIP_PITCH: limit lower=-3.14 upper=1.8 effort=30 velocity=13.0 -> (none)
- joint FL_HIP_ROLL: limit lower=-1.8 upper=1.8 effort=30 velocity=13.0 -> (none)
- joint FL_KNEE_PITCH: limit lower=-3.14 upper=0.0 effort=30 velocity=13.0 -> (none)
